File: hardware/capture/chipwhisperer-lite/pcb/eagle/cw-lite-main.brd (EAGLE design)
At the start: 117 x 60 mm, 290 parts, among them J1 SHROUD_2X10-SHROUDED, J2 SHROUD_2X10-SHROUDED, J3 SHROUD_2X10-SHROUDED, J4 CON_HEADER_PRG_XILINX_JTAG6, J5 PINHD-1X10, J6 SHROUD_2X4SHROUD, J7 SHROUD_2X4EDGE, J8 MICRO-USB-5P-ZX62D-B-5P8, J9 MICRO-USB-5P-ZX62D-B-5P8, T1 IRLML6402TRPBF, T2 IRLML2502, T3 IRLML6402TRPBF, T4 IRLML2502, U1 ATSAM3U2CA-AU, U10 LP3985IM5-3.0, U11 V_REG_MIC2920, U12 XMEGA128A4U, U2 6SLX9TQG144, U3 AD8331, U4 AD9215BRUZ, U5 LTC3419EMS, U6 PRTR5V0U2AX, U7 TC1262-3.3VDBTR, U8 IRF7807ZTRPBF, U9 SPI_FLASH-X25XXSMD1, X2 SMA-NOSILK, X3 SMA-NOSILK, X4 SMA-NOSILK, X5 SMA-NOSILK

Commit message: version without target part
Parts:
- removed C103: 10u, custom-std:0603C
- removed C104: 10n, custom-std:0603C
- removed C105, C107: 1u, custom-std:0603C
- removed C106, C108, C109: 100n, custom-std:0603C
- removed C115, C116, C121: DNM, custom-std:0603C
- removed C118, C119, C120: (no value), custom-std:0603C
- removed C37: 47u, custom-std:0805
- removed J2: SHROUD_2X10-SHROUDED, custom-std:PINSHRD_PTH_2X10
- removed J9: MICRO-USB-5P-ZX62D-B-5P8, customs:B-SMD-5P-TH
- removed JP12, JP6, JP7: (no value), pinhead:1X02
- removed JP13: (no value), adafruit:1X09-BIG
- removed JP14, JP15, JP16, JP17: (no value), adafruit:1X01
- removed L10: 1k/500mA, dp_devices:FB603
- removed LED10, LED9: (no value), dp_devices:LED-603
- removed Q2: (no value), crystal:HC49U-V
- removed R13: 10k, custom-std:0603R
- removed R66, R76: 49R9, custom-std:0805
- removed R67, R72: 100R, custom-std:0603R
- removed R73: DNM, custom-std:0603R
- removed R74, R75: 1k, custom-std:0603R
- removed SJ2: (no value), SparkFun:SJ_3_PASTE2&3
- removed SJ3, SJ4, SJ5, SJ7: SOLDERJUMPERNC, SparkFun:SJ_2S
- removed U11: V_REG_MIC2920, SparkFun-PowerIC:SOT223
- removed U12: XMEGA128A4U, atmel:TQFP44
- removed X3, X5: SMA-NOSILK, custom-std:J502-ND-142-0711-821/826-NOSILK
Connections:
- removed net N$111: C105.1, C106.1, C37.1, JP12.2, R76.1, SJ3.1
- removed net N$14: C118.2, J9.E1, J9.E2, J9.P$1, J9.P$2, J9.P$3, J9.P$4
- removed net N$39: C107.1, C108.1, C109.2, JP12.1, R66.2, SJ3.2, U12.39
- removed net N$43: C121.2, JP6.1, JP7.1, R66.1, SJ4.1, SJ5.1, U12.19, U12.31, U12.9
- removed net N$44: C119.2, J9.1, U11.1
- removed net N$46: C120.2, SJ2.1, U11.3
- removed net N$47: LED9.A, R74.1
- removed net N$48: LED10.A, R75.1
- removed net N$50: LED9.C, U12.1
- removed net N$51: LED10.C, U12.2
- removed net N$52: JP13.1, U12.25
- removed net N$53: JP13.2, U12.24
- removed net N$54: JP13.3, U12.23
- removed net N$55: JP13.4, U12.22
- removed net N$56: JP13.5, U12.21
- removed net N$57: C115.1, Q2.2, R72.1, U12.37
- removed net N$58: C116.2, Q2.1, R73.1, U12.36
- removed net N$59: R67.2, U12.7
- removed net N$60: JP13.6, U12.20
- removed net N$61: L10.2, R76.2
- removed net TPC6: JP13.8, U12.16
- removed net TPC7: JP13.7, U12.17
- removed net TUSB_N: J9.2, U12.26
- removed net TUSB_P: J9.3, U12.27
- removed net VCC_TARG: C103.1, C104.1, L10.1, R13.1, R74.2, R75.2, SJ2.2, SJ7.1
- net ANIN: no longer JP7.2, SJ4.2, X3.1
- net GND: no longer C103.2, C104.2, C105.2, C106.2, C107.2, C108.2, C109.1, C115.2, C116.1, C118.1, C119.1, C120.1, C121.1, C37.2, J2.17, J2.19, J2.2, J9.5, JP13.9, U11.2, U12.18, U12.30, U12.38, U12.8, X3.G@1, X3.G@2, X3.G@3, X3.G@4, X5.G@1, X5.G@2, X5.G@3, X5.G@4
- net THS1: no longer J2.4, R67.1
- net THS2: no longer J2.6, R72.2, R73.2
- net TIO1: no longer J2.10, JP16.1, U12.13
- net TIO2: no longer J2.12, JP17.1, U12.12
- net TIO3: no longer J2.14, JP14.1, U12.41
- net TIO4: no longer J2.16, JP15.1, U12.40
- net TMISO: no longer J2.7
- net TMOSI: no longer J2.9
- net TPDIC: no longer J2.13, R13.2, U12.35
- net TPDID: no longer J2.15, U12.34
- net TRST: no longer J2.5
- net TSCK: no longer J2.11
- net TVREF: no longer J2.8, SJ7.2
- net VCCGLITCH: no longer JP6.2, SJ5.2, X5.1
- net VCCTIO_SWITCHED: no longer J2.18, J2.3, SJ2.3
Routing:
- net GND: track 644.6 -> 394.3 mm, vias 280 -> 229
- net VCCTIO_SWITCHED: track 178.5 -> 71.8 mm, vias 7 -> 2
- net VCC_TARG: track 92.0 -> 0.00 mm, vias 5 -> 0
- net TPDIC: track 95.1 -> 34.1 mm, vias 3 -> 1
- net N$43: track 60.3 -> 0.00 mm, vias 2 -> 0
- net N$39: track 46.2 -> 0.00 mm, vias 2 -> 0
- net TIO2: track 71.1 -> 28.8 mm, vias 1 -> 0
- net N$46: track 41.8 -> 0.00 mm, vias 2 -> 0
- net TIO1: track 69.9 -> 28.5 mm, vias 1 -> 0
- net N$52: track 40.0 -> 0.00 mm, vias 2 -> 0
- net TPDID: track 80.0 -> 42.5 mm, vias 5 -> 3
- net N$53: track 36.6 -> 0.00 mm, vias 2 -> 0
- net N$54: track 35.5 -> 0.00 mm, vias 2 -> 0
- net TIO3: track 60.3 -> 27.8 mm
- net TPC6: track 29.5 -> 0.00 mm, vias 1 -> 0
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Other:
- board size 117 x 60 mm -> 82.1 x 60 mm
- board text removed: "+3.3V"
- board text removed: "Also 16/32/64 fit in TQ44"
- board text removed: "DEVICE UNDER TEST"
- board text removed: "IDC"
- board text removed: "IN"
- board text removed: "OUT"
- board text removed: "PC6"
- board text removed: "PC7"
- board text removed: "PD0"
- board text removed: "PD1"
- board text removed: "PD2"
- board text removed: "PD3"
- board text removed: "PD4"
- board text removed: "PD5"
- board text removed: "RXD"
- board text removed: "Suggested area to add board ID / Logos on bottom silkscreen layer"
- board text removed: "TIO1"
- board text removed: "TIO2"
- board text removed: "TIO3"
- board text removed: "TIO4"
- board text removed: "TXD"
- board text removed: "These unplated holes for allowing seperating sections of PCBs. Normally PCBs are attached so traces routed between holes are required, please manufacture AS-IS."
- board text removed: "X1"
- board text removed: "X2"
- board text removed: "XMEGA128A4U"
