File: hardware/capture/chipwhisperer-lite/pcb/eagle/cw-lite-main.sch (EAGLE design)
At the start: 290 parts, among them J1 SHROUD_2X10-SHROUDED, J2 SHROUD_2X10-SHROUDED, J3 SHROUD_2X10-SHROUDED, J4 CON_HEADER_PRG_XILINX_JTAG6, J5 PINHD-1X10, J6 SHROUD_2X4SHROUD, J7 SHROUD_2X4EDGE, J8 MICRO-USB-5P-ZX62D-B-5P8, J9 MICRO-USB-5P-ZX62D-B-5P8, T1 IRLML6402TRPBF, T2 IRLML2502, T3 IRLML6402TRPBF, T4 IRLML2502, U1 ATSAM3U2CA-AU, U10 LP3985IM5-3.0, U11 V_REG_MIC2920, U12 XMEGA128A4U, U2 6SLX9TQG144, U3 AD8331, U4 AD9215BRUZ, U5 LTC3419EMS, U6 PRTR5V0U2AX, U7 TC1262-3.3VDBTR, U8 IRF7807ZTRPBF, U9 SPI_FLASH-X25XXSMD1, X2 SMA-NOSILK, X3 SMA-NOSILK, X4 SMA-NOSILK, X5 SMA-NOSILK

Commit message: version without target part
Parts:
- removed C103: 10u, custom-std:CAP0603-CAP
- removed C104: 10n, custom-std:CAP0603-CAP
- removed C105, C107: 1u, custom-std:CAP0603-CAP
- removed C106, C108, C109: 100n, custom-std:CAP0603-CAP
- removed C115, C116, C121: DNM, custom-std:CAP0603-CAP
- removed C118, C119, C120: (no value), custom-std:CAP0603-CAP
- removed C37: 47u, custom-std:CAP0805
- removed J2: SHROUD_2X10-SHROUDED, custom-std:SHROUD_2X10-SHROUDED
- removed J9: MICRO-USB-5P-ZX62D-B-5P8, customs:MICRO-USB-5P-ZX62D-B-5P8
- removed JP12, JP6, JP7: (no value), pinhead:PINHD-1X2
- removed JP13: (no value), adafruit:PINHD-1X9
- removed JP14, JP15, JP16, JP17: (no value), adafruit:PINHD-1X1
- removed L10: 1k/500mA, dp_devices:FERRITE-0603
- removed LED10, LED9: (no value), dp_devices:LED-0603
- removed Q2: (no value), crystal:CRYSTALHC49U-V
- removed R13: 10k, custom-std:RES0603-RES
- removed R66, R76: 49R9, custom-std:RES0805-RES
- removed R67, R72: 100R, custom-std:RES0603-RES
- removed R73: DNM, custom-std:RES0603-RES
- removed R74, R75: 1k, custom-std:RES0603-RES
- removed SJ2: (no value), SparkFun:SOLDERJUMPER_2WAYPASTE2&3
- removed SJ3, SJ4, SJ5, SJ7: SOLDERJUMPERNC, SparkFun:SOLDERJUMPERNC
- removed U11: V_REG_MIC2920, SparkFun-PowerIC:V_REG_MIC2920
- removed U12: XMEGA128A4U, atmel:XMEGA16A4A
- removed X3, X5: SMA-NOSILK, custom-std:SMA-NOSILK
Connections:
- removed net N$111: C105.1, C106.1, C37.1, JP12.2, R76.1, SJ3.1
- removed net N$14: C118.2, J9.SHIELD
- removed net N$39: C107.1, C108.1, C109.2, JP12.1, R66.2, SJ3.2, U12.AVCC
- removed net N$43: C121.2, JP6.1, JP7.1, R66.1, SJ4.1, SJ5.1, U12.VCC, U12.VCC1, U12.VCC2
- removed net N$44: C119.2, J9.VCC, U11.IN
- removed net N$46: C120.2, SJ2.1, U11.OUT
- removed net N$47: LED9.A, R74.1
- removed net N$48: LED10.A, R75.1
- removed net N$50: LED9.C, U12.PA5
- removed net N$51: LED10.C, U12.PA6
- removed net N$52: JP13.1, U12.PD5
- removed net N$53: JP13.2, U12.PD4
- removed net N$54: JP13.3, U12.PD3
- removed net N$55: JP13.4, U12.PD2
- removed net N$56: JP13.5, U12.PD1
- removed net N$57: C115.1, Q2.2, R72.1, U12.PR1(XT1)
- removed net N$58: C116.2, Q2.1, R73.1, U12.PR0(XT2)
- removed net N$59: R67.2, U12.PB3
- removed net N$60: JP13.6, U12.PD0
- removed net N$61: L10.2, R76.2
- removed net TPC6: JP13.8, U12.PC6
- removed net TPC7: JP13.7, U12.PC7
- removed net TUSB_N: J9.DM, U12.PD6
- removed net TUSB_P: J9.DP, U12.PD7
- removed net VCC_TARG: C103.1, C104.1, L10.1, R13.1, R74.2, R75.2, SJ2.2, SJ7.1
- net ANIN: no longer JP7.2, SJ4.2, X3.1
- net GND: no longer C103.2, C104.2, C105.2, C106.2, C107.2, C108.2, C109.1, C115.2, C116.1, C118.1, C119.1, C120.1, C121.1, C37.2, J2.17, J2.19, J2.2, J9.GND@1, JP13.9, U11.GND, U12.GND, U12.GND1, U12.GND2, U12.GND3, X3.2, X5.2
- net THS1: no longer J2.4, R67.1
- net THS2: no longer J2.6, R72.2, R73.2
- net TIO1: no longer J2.10, JP16.1, U12.PC3
- net TIO2: no longer J2.12, JP17.1, U12.PC2
- net TIO3: no longer J2.14, JP14.1, U12.PA1
- net TIO4: no longer J2.16, JP15.1, U12.PA0
- net TMISO: no longer J2.7
- net TMOSI: no longer J2.9
- net TPDIC: no longer J2.13, R13.2, U12.!RESET!/PDI_CLK
- net TPDID: no longer J2.15, U12.PDI_DATA
- net TRST: no longer J2.5
- net TSCK: no longer J2.11
- net TVREF: no longer J2.8, SJ7.2
- net VCCGLITCH: no longer JP6.2, SJ5.2, X5.1
- net VCCTIO_SWITCHED: no longer J2.18, J2.3, SJ2.3
Other:
- note removed: "Breakaway Section of PCB"
- note removed: "Might be XMEGA128D3 instead?"
